File: lightrailwww.kicad_pcb (KiCad board)
At the start: 16 copper layers, 95 x 82 mm, 18 parts, among them J1 Conn_01x03, J2 Conn_02x10_Counter_Clockwise, J3 Conn_02x18_Counter_Clockwise, J4 Conn_02x06_Counter_Clockwise, J5 Conn_01x04, J6 Conn_02x05_Counter_Clockwise, U1 AMS1117-3.3, U2 AMS1117-1.8, U3 W25Q128JVE, U4 LMV358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

Commit message: Update PCB stackup to 6 copper layers as requested by fab
Routing:
- net (no net): track 1050.7 -> 1350.9 mm
- added copper zone on In1.Cu, net unconnected-(J3-Pin_19-Pad19)
- added copper zone on In2.Cu, net unconnected-(J3-Pin_19-Pad19)
- added copper zone on In3.Cu, net unconnected-(J3-Pin_19-Pad19)
- added copper zone on In4.Cu, net unconnected-(J3-Pin_19-Pad19)
- removed copper zone on In13.Cu, net unconnected-(J3-Pin_12-Pad12)
- removed copper zone on In14.Cu, net unconnected-(J3-Pin_12-Pad12)
Other:
- copper layers 16 -> 6
Changed lines of the file:
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@@
 		(8 "In3.Cu" signal)
 		(10 "In4.Cu" signal)
-		(12 "In5.Cu" signal)
-		(14 "In6.Cu" signal)
-		(16 "In7.Cu" signal)
-		(18 "In8.Cu" signal)
-		(20 "In9.Cu" signal)
-		(22 "In10.Cu" signal)
-		(24 "In11.Cu" signal)
-		(26 "In12.Cu" signal)
-		(28 "In13.Cu" signal)
-		(30 "In14.Cu" signal)
 		(2 "B.Cu" signal)
 		(9 "F.Adhes" user "F.Adhesive")
@@
 		(end 170.025 73.975)
 		(width 0.25)
+		(layer "In1.Cu")
+		(net 0)
+	)
+	(segment
+		(start 94.975 73.975)
+		(end 170.025 73.975)
+		(width 0.25)
 		(layer "In2.Cu")
 		(net 0)
@@
 		(end 170.025 73.975)
 		(width 0.25)
+		(layer "In2.Cu")
+		(net 0)
+	)
+	(segment
+		(start 94.975 73.975)
+		(end 170.025 73.975)
+		(width 0.25)
+		(layer "In3.Cu")
+		(net 0)
+	)
+	(segment
+		(start 94.975 73.975)
+		(end 170.025 73.975)
+		(width 0.25)
 		(layer "In3.Cu")
 		(net 0)
@@
 		(end 170.025 73.975)
 		(width 0.25)
+		(layer "In4.Cu")
+		(net 0)
+	)
+	(segment
+		(start 94.975 73.975)
+		(end 170.025 73.975)
+		(width 0.25)
 		(layer "In5.Cu")
 		(net 0)
@@
 	)
 	(zone
+		(net 35)
+		(net_name "unconnected-(J3-Pin_19-Pad19)")
+		(layer "In1.Cu")
+		(hatch edge 0.5)
+		(connect_pads
+			(clearance 0.5)
+		)
+		(min_thickness 0.25)
+		(filled_areas_thickness no)
+		(fill yes
+			(thermal_gap 0.5)
+			(thermal_bridge_width 0.5)
+		)
+		(polygon
+			(pts
+				(xy 84.975 63.975) (xy 180.025 63.975) (xy 180.025 146.025) (xy 84.975 146.025)
+			)
+		)
+	)
+	(zone
+		(net 35)
+		(net_name "unconnected-(J3-Pin_19-Pad19)")
+		(layer "In2.Cu")
+		(hatch edge 0.5)
+		(connect_pads
+			(clearance 0.5)
+		)
+		(min_thickness 0.25)
+		(filled_areas_thickness no)
+		(fill yes
+			(thermal_gap 0.5)
+			(thermal_bridge_width 0.5)
+		)
+		(polygon
+			(pts
+				(xy 84.975 63.975) (xy 180.025 63.975) (xy 180.025 146.025) (xy 84.975 146.025)
+			)
+		)
+	)
+	(zone
 		(net 36)
 		(net_name "unconnected-(J3-Pin_12-Pad12)")
@@
 		(hatch edge 0.5)
 		(connect_pads
+			(clearance 0.5)
+		)
+		(min_thickness 0.25)
+		(filled_areas_thickness no)
+		(fill yes
+			(thermal_gap 0.5)
+			(thermal_bridge_width 0.5)
+		)
+		(polygon
+			(pts
+				(xy 84.975 63.975) (xy 180.025 63.975) (xy 180.025 146.025) (xy 84.975 146.025)
+			)
+		)
+	)
+	(zone
+		(net 35)
+		(net_name "unconnected-(J3-Pin_19-Pad19)")
+		(layer "In3.Cu")
+		(hatch edge 0.5)
+		(connect_pads
+			(clearance 0.5)
+		)
+		(min_thickness 0.25)
+		(filled_areas_thickness no)
+		(fill yes
+			(thermal_gap 0.5)
+			(thermal_bridge_width 0.5)
+		)
+		(polygon
+			(pts
+				(xy 84.975 63.975) (xy 180.025 63.975) (xy 180.025 146.025) (xy 84.975 146.025)
+			)
+		)
+	)
+	(zone
+		(net 35)
+		(net_name "unconnected-(J3-Pin_19-Pad19)")
+		(layer "In4.Cu")
+		(hatch edge 0.5)
+		(connect_pads

Commit message: Revert "Update PCB stackup to 6 copper layers as requested by fab"
This reverts commit 9de2d115b8448442437ad79354c111fe7e6ef276.
Routing:
- net (no net): track 1350.9 -> 1050.7 mm
- added copper zone on In13.Cu, net unconnected-(J3-Pin_12-Pad12)
- added copper zone on In14.Cu, net unconnected-(J3-Pin_12-Pad12)
- removed copper zone on In1.Cu, net unconnected-(J3-Pin_19-Pad19)
- removed copper zone on In2.Cu, net unconnected-(J3-Pin_19-Pad19)
- removed copper zone on In3.Cu, net unconnected-(J3-Pin_19-Pad19)
- removed copper zone on In4.Cu, net unconnected-(J3-Pin_19-Pad19)
Other:
- copper layers 6 -> 16
Changed lines of the file:
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@@
 		(8 "In3.Cu" signal)
 		(10 "In4.Cu" signal)
+		(12 "In5.Cu" signal)
+		(14 "In6.Cu" signal)
+		(16 "In7.Cu" signal)
+		(18 "In8.Cu" signal)
+		(20 "In9.Cu" signal)
+		(22 "In10.Cu" signal)
+		(24 "In11.Cu" signal)
+		(26 "In12.Cu" signal)
+		(28 "In13.Cu" signal)
+		(30 "In14.Cu" signal)
 		(2 "B.Cu" signal)
 		(9 "F.Adhes" user "F.Adhesive")
@@
 		(end 170.025 73.975)
 		(width 0.25)
-		(layer "In1.Cu")
-		(net 0)
-	)
-	(segment
-		(start 94.975 73.975)
-		(end 170.025 73.975)
-		(width 0.25)
 		(layer "In2.Cu")
 		(net 0)
@@
 		(end 170.025 73.975)
 		(width 0.25)
-		(layer "In2.Cu")
-		(net 0)
-	)
-	(segment
-		(start 94.975 73.975)
-		(end 170.025 73.975)
-		(width 0.25)
-		(layer "In3.Cu")
-		(net 0)
-	)
-	(segment
-		(start 94.975 73.975)
-		(end 170.025 73.975)
-		(width 0.25)
 		(layer "In3.Cu")
 		(net 0)
@@
 		(end 170.025 73.975)
 		(width 0.25)
-		(layer "In4.Cu")
-		(net 0)
-	)
-	(segment
-		(start 94.975 73.975)
-		(end 170.025 73.975)
-		(width 0.25)
 		(layer "In5.Cu")
 		(net 0)
@@
 	)
 	(zone
-		(net 35)
-		(net_name "unconnected-(J3-Pin_19-Pad19)")
-		(layer "In1.Cu")
-		(hatch edge 0.5)
-		(connect_pads
-			(clearance 0.5)
-		)
-		(min_thickness 0.25)
-		(filled_areas_thickness no)
-		(fill yes
-			(thermal_gap 0.5)
-			(thermal_bridge_width 0.5)
-		)
-		(polygon
-			(pts
-				(xy 84.975 63.975) (xy 180.025 63.975) (xy 180.025 146.025) (xy 84.975 146.025)
-			)
-		)
-	)
-	(zone
-		(net 35)
-		(net_name "unconnected-(J3-Pin_19-Pad19)")
-		(layer "In2.Cu")
-		(hatch edge 0.5)
-		(connect_pads
-			(clearance 0.5)
-		)
-		(min_thickness 0.25)
-		(filled_areas_thickness no)
-		(fill yes
-			(thermal_gap 0.5)
-			(thermal_bridge_width 0.5)
-		)
-		(polygon
-			(pts
-				(xy 84.975 63.975) (xy 180.025 63.975) (xy 180.025 146.025) (xy 84.975 146.025)
-			)
-		)
-	)
-	(zone
 		(net 36)
 		(net_name "unconnected-(J3-Pin_12-Pad12)")
@@
 		(hatch edge 0.5)
 		(connect_pads
-			(clearance 0.5)
-		)
-		(min_thickness 0.25)
-		(filled_areas_thickness no)
-		(fill yes
-			(thermal_gap 0.5)
-			(thermal_bridge_width 0.5)
-		)
-		(polygon
-			(pts
-				(xy 84.975 63.975) (xy 180.025 63.975) (xy 180.025 146.025) (xy 84.975 146.025)
-			)
-		)
-	)
-	(zone
-		(net 35)
-		(net_name "unconnected-(J3-Pin_19-Pad19)")
-		(layer "In3.Cu")
-		(hatch edge 0.5)
-		(connect_pads
-			(clearance 0.5)
-		)
-		(min_thickness 0.25)
-		(filled_areas_thickness no)
-		(fill yes
-			(thermal_gap 0.5)
-			(thermal_bridge_width 0.5)
-		)
-		(polygon
-			(pts
-				(xy 84.975 63.975) (xy 180.025 63.975) (xy 180.025 146.025) (xy 84.975 146.025)
-			)
-		)
-	)
-	(zone
-		(net 35)
-		(net_name "unconnected-(J3-Pin_19-Pad19)")
-		(layer "In4.Cu")
-		(hatch edge 0.5)
-		(connect_pads
