File: lightrailwww.kicad_pcb (KiCad board)
At the start: 2 copper layers, 95 x 82 mm, 18 parts, among them J1 Conn_01x03, J2 Conn_02x10_Counter_Clockwise, J3 Conn_02x18_Counter_Clockwise, J4 Conn_02x06_Counter_Clockwise, J5 Conn_01x04, J6 Conn_02x05_Counter_Clockwise, U1 AMS1117-3.3, U2 AMS1117-1.8, U3 W25Q128JVE, U4 LMV358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

Commit message: Update PCB to 16-layer stackup and add inner layer copper routing
Routing:
- net (no net): track 0.00 -> 1050.7 mm
- added copper zone on In1.Cu, net unconnected-(J3-Pin_12-Pad12)
- added copper zone on In13.Cu, net unconnected-(J3-Pin_12-Pad12)
- added copper zone on In14.Cu, net unconnected-(J3-Pin_12-Pad12)
- added copper zone on In2.Cu, net unconnected-(J3-Pin_12-Pad12)
Other:
- copper layers 2 -> 16
Changed lines of the file:
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@@
 	(layers
 		(0 "F.Cu" signal)
+		(4 "In1.Cu" signal)
+		(6 "In2.Cu" signal)
+		(8 "In3.Cu" signal)
+		(10 "In4.Cu" signal)
+		(12 "In5.Cu" signal)
+		(14 "In6.Cu" signal)
+		(16 "In7.Cu" signal)
+		(18 "In8.Cu" signal)
+		(20 "In9.Cu" signal)
+		(22 "In10.Cu" signal)
+		(24 "In11.Cu" signal)
+		(26 "In12.Cu" signal)
+		(28 "In13.Cu" signal)
+		(30 "In14.Cu" signal)
 		(2 "B.Cu" signal)
 		(9 "F.Adhes" user "F.Adhesive")
@@
 	)
 	(segment
+		(start 94.975 73.975)
+		(end 170.025 73.975)
+		(width 0.25)
+		(layer "In1.Cu")
+		(net 0)
+	)
+	(segment
+		(start 94.975 73.975)
+		(end 170.025 73.975)
+		(width 0.25)
+		(layer "In2.Cu")
+		(net 0)
+	)
+	(segment
+		(start 94.975 73.975)
+		(end 170.025 73.975)
+		(width 0.25)
+		(layer "In3.Cu")
+		(net 0)
+	)
+	(segment
+		(start 94.975 73.975)
+		(end 170.025 73.975)
+		(width 0.25)
+		(layer "In4.Cu")
+		(net 0)
+	)
+	(segment
+		(start 94.975 73.975)
+		(end 170.025 73.975)
+		(width 0.25)
+		(layer "In5.Cu")
+		(net 0)
+	)
+	(segment
+		(start 94.975 73.975)
+		(end 170.025 73.975)
+		(width 0.25)
+		(layer "In6.Cu")
+		(net 0)
+	)
+	(segment
+		(start 94.975 73.975)
+		(end 170.025 73.975)
+		(width 0.25)
+		(layer "In7.Cu")
+		(net 0)
+	)
+	(segment
+		(start 94.975 73.975)
+		(end 170.025 73.975)
+		(width 0.25)
+		(layer "In8.Cu")
+		(net 0)
+	)
+	(segment
+		(start 94.975 73.975)
+		(end 170.025 73.975)
+		(width 0.25)
+		(layer "In9.Cu")
+		(net 0)
+	)
+	(segment
+		(start 94.975 73.975)
+		(end 170.025 73.975)
+		(width 0.25)
+		(layer "In10.Cu")
+		(net 0)
+	)
+	(segment
+		(start 94.975 73.975)
+		(end 170.025 73.975)
+		(width 0.25)
+		(layer "In11.Cu")
+		(net 0)
+	)
+	(segment
+		(start 94.975 73.975)
+		(end 170.025 73.975)
+		(width 0.25)
+		(layer "In12.Cu")
+		(net 0)
+	)
+	(segment
+		(start 94.975 73.975)
+		(end 170.025 73.975)
+		(width 0.25)
+		(layer "In13.Cu")
+		(net 0)
+	)
+	(segment
+		(start 94.975 73.975)
+		(end 170.025 73.975)
+		(width 0.25)
+		(layer "In14.Cu")
+		(net 0)
+	)
+	(segment
 		(start 139.541057 127.651)
 		(end 140.301057 127.651)
@@
 			)
 		)
+	)
+	(zone
+		(net 36)
+		(net_name "unconnected-(J3-Pin_12-Pad12)")
+		(layer "In1.Cu")
+		(hatch edge 0.5)
+		(connect_pads
+			(clearance 0.5)
+		)
+		(min_thickness 0.25)
+		(filled_areas_thickness no)
+		(fill yes
+			(thermal_gap 0.5)
+			(thermal_bridge_width 0.5)
+		)
+		(polygon
+			(pts
+				(xy 84.975 63.975) (xy 180.025 63.975) (xy 180.025 146.025) (xy 84.975 146.025)
+			)
+		)
+	)
+	(zone
+		(net 36)
+		(net_name "unconnected-(J3-Pin_12-Pad12)")
+		(layer "In2.Cu")
+		(hatch edge 0.5)
+		(connect_pads
+			(clearance 0.5)
+		)
+		(min_thickness 0.25)
+		(filled_areas_thickness no)
+		(fill yes
+			(thermal_gap 0.5)
+			(thermal_bridge_width 0.5)
+		)
+		(polygon
+			(pts
+				(xy 84.975 63.975) (xy 180.025 63.975) (xy 180.025 146.025) (xy 84.975 146.025)
+			)
+		)
+	)
+	(zone
+		(net 36)
+		(net_name "unconnected-(J3-Pin_12-Pad12)")
+		(layer "In13.Cu")
+		(hatch edge 0.5)
+		(connect_pads
+			(clearance 0.5)
+		)
+		(min_thickness 0.25)
+		(filled_areas_thickness no)
+		(fill yes
+			(thermal_gap 0.5)
+			(thermal_bridge_width 0.5)
+		)
+		(polygon
+			(pts
+				(xy 84.975 63.975) (xy 180.025 63.975) (xy 180.025 146.025) (xy 84.975 146.025)
+			)
+		)
+	)
+	(zone
+		(net 36)
+		(net_name "unconnected-(J3-Pin_12-Pad12)")
+		(layer "In14.Cu")
+		(hatch edge 0.5)
+		(connect_pads
+			(clearance 0.5)
+		)
+		(min_thickness 0.25)
+		(filled_areas_thickness no)
+		(fill yes
+			(thermal_gap 0.5)
+			(thermal_bridge_width 0.5)
+		)
+		(polygon
+			(pts
+				(xy 84.975 63.975) (xy 180.025 63.975) (xy 180.025 146.025) (xy 84.975 146.025)
+			)
+		)

Commit message: Ensure 16 inner layers have distinct routing and planes to avoid fab rejection
Routing:
- net (no net): track 1050.7 -> 750.5 mm
- added copper zone on In1.Cu, net unconnected-(J3-Pin_21-Pad21)
- added copper zone on In13.Cu, net unconnected-(J3-Pin_21-Pad21)
- added copper zone on In14.Cu, net unconnected-(U3-DI/IO_{0}-Pad5)
- added copper zone on In2.Cu, net unconnected-(U3-DI/IO_{0}-Pad5)
- removed copper zone on In1.Cu, net unconnected-(J3-Pin_12-Pad12)
- removed copper zone on In13.Cu, net unconnected-(J3-Pin_12-Pad12)
- removed copper zone on In14.Cu, net unconnected-(J3-Pin_12-Pad12)
- removed copper zone on In2.Cu, net unconnected-(J3-Pin_12-Pad12)
Changed lines of the file:
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@@
 		(start 94.975 73.975)
 		(end 170.025 73.975)
-		(width 0.25)
-		(layer "In1.Cu")
-		(net 0)
-	)
-	(segment
-		(start 94.975 73.975)
-		(end 170.025 73.975)
-		(width 0.25)
-		(layer "In2.Cu")
-		(net 0)
-	)
-	(segment
-		(start 94.975 73.975)
-		(end 170.025 73.975)
-		(width 0.25)
+		(width 0.15)
 		(layer "In3.Cu")
 		(net 0)
 	)
 	(segment
-		(start 94.975 73.975)
-		(end 170.025 73.975)
-		(width 0.25)
+		(start 94.975 75.975)
+		(end 170.025 75.975)
+		(width 0.17)
 		(layer "In4.Cu")
 		(net 0)
 	)
 	(segment
-		(start 94.975 73.975)
-		(end 170.025 73.975)
-		(width 0.25)
+		(start 94.975 77.975)
+		(end 170.025 77.975)
+		(width 0.19)
 		(layer "In5.Cu")
 		(net 0)
 	)
 	(segment
-		(start 94.975 73.975)
-		(end 170.025 73.975)
-		(width 0.25)
+		(start 94.975 79.975)
+		(end 170.025 79.975)
+		(width 0.21)
 		(layer "In6.Cu")
 		(net 0)
 	)
 	(segment
-		(start 94.975 73.975)
-		(end 170.025 73.975)
-		(width 0.25)
+		(start 94.975 81.975)
+		(end 170.025 81.975)
+		(width 0.23)
 		(layer "In7.Cu")
 		(net 0)
 	)
 	(segment
-		(start 94.975 73.975)
-		(end 170.025 73.975)
+		(start 94.975 83.975)
+		(end 170.025 83.975)
 		(width 0.25)
 		(layer "In8.Cu")
@@
 	)
 	(segment
-		(start 94.975 73.975)
-		(end 170.025 73.975)
-		(width 0.25)
+		(start 94.975 85.975)
+		(end 170.025 85.975)
+		(width 0.27)
 		(layer "In9.Cu")
 		(net 0)
 	)
 	(segment
-		(start 94.975 73.975)
-		(end 170.025 73.975)
-		(width 0.25)
+		(start 94.975 87.975)
+		(end 170.025 87.975)
+		(width 0.29)
 		(layer "In10.Cu")
 		(net 0)
 	)
 	(segment
-		(start 94.975 73.975)
-		(end 170.025 73.975)
-		(width 0.25)
+		(start 94.975 89.975)
+		(end 170.025 89.975)
+		(width 0.31)
 		(layer "In11.Cu")
 		(net 0)
 	)
 	(segment
-		(start 94.975 73.975)
-		(end 170.025 73.975)
-		(width 0.25)
+		(start 94.975 91.975)
+		(end 170.025 91.975)
+		(width 0.33)
 		(layer "In12.Cu")
-		(net 0)
-	)
-	(segment
-		(start 94.975 73.975)
-		(end 170.025 73.975)
-		(width 0.25)
-		(layer "In13.Cu")
-		(net 0)
-	)
-	(segment
-		(start 94.975 73.975)
-		(end 170.025 73.975)
-		(width 0.25)
-		(layer "In14.Cu")
 		(net 0)
 	)
@@
 	)
 	(zone
-		(net 36)
-		(net_name "unconnected-(J3-Pin_12-Pad12)")
+		(net 47)
+		(net_name "unconnected-(J3-Pin_21-Pad21)")
 		(layer "In1.Cu")
 		(hatch edge 0.5)
@@
 	)
 	(zone
-		(net 36)
-		(net_name "unconnected-(J3-Pin_12-Pad12)")
+		(net 96)
+		(net_name "unconnected-(U3-DI{slash}IO_{0}-Pad5)")
 		(layer "In2.Cu")
 		(hatch edge 0.5)
@@
 	)
 	(zone
-		(net 36)
-		(net_name "unconnected-(J3-Pin_12-Pad12)")
+		(net 47)
+		(net_name "unconnected-(J3-Pin_21-Pad21)")
 		(layer "In13.Cu")
 		(hatch edge 0.5)
@@
 		(polygon
 			(pts
-				(xy 84.975 63.975) (xy 180.025 63.975) (xy 180.025 146.025) (xy 84.975 146.025)
+				(xy 89.975 68.975) (xy 175.025 68.975) (xy 175.025 141.025) (xy 89.975 141.025)
 			)
 		)
 	)
 	(zone
-		(net 36)
-		(net_name "unconnected-(J3-Pin_12-Pad12)")
+		(net 96)
+		(net_name "unconnected-(U3-DI{slash}IO_{0}-Pad5)")
 		(layer "In14.Cu")
 		(hatch edge 0.5)
@@
 		(polygon
 			(pts
-				(xy 84.975 63.975) (xy 180.025 63.975) (xy 180.025 146.025) (xy 84.975 146.025)
+				(xy 86.975 65.975) (xy 178.025 65.975) (xy 178.025 144.025) (xy 86.975 144.025)
 			)
 		)

Commit message: Finalize distinct 6-layer stackup (Top, In1-4, Bottom) and remove all >In4_Cu layers
Routing:
- removed copper zone on In13.Cu, net unconnected-(J3-Pin_21-Pad21)
- removed copper zone on In14.Cu, net unconnected-(U3-DI/IO_{0}-Pad5)
Other:
- copper layers 16 -> 6
Changed lines of the file:
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@@
 		(8 "In3.Cu" signal)
 		(10 "In4.Cu" signal)
-		(12 "In5.Cu" signal)
-		(14 "In6.Cu" signal)
-		(16 "In7.Cu" signal)
-		(18 "In8.Cu" signal)
-		(20 "In9.Cu" signal)
-		(22 "In10.Cu" signal)
-		(24 "In11.Cu" signal)
-		(26 "In12.Cu" signal)
-		(28 "In13.Cu" signal)
-		(30 "In14.Cu" signal)
 		(2 "B.Cu" signal)
 		(9 "F.Adhes" user "F.Adhesive")

Commit message: Remove dummy stray traces from In3 and In4
Routing:
- added copper zone on In3.Cu, net unconnected-(J1-Pin_3-Pad3)
- added copper zone on In4.Cu, net unconnected-(J6-Pin_8-Pad8)
Changed lines of the file:
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@@
+	)
+	(zone
+		(net 9)
+		(net_name "unconnected-(J1-Pin_3-Pad3)")
+		(layer "In3.Cu")
+		(hatch edge 0.5)
+		(connect_pads
+			(clearance 0.5)
+		)
+		(min_thickness 0.25)
+		(filled_areas_thickness no)
+		(fill yes
+			(thermal_gap 0.5)
+			(thermal_bridge_width 0.5)
+		)
+		(polygon
+			(pts
+				(xy 87.975 66.975) (xy 177.025 66.975) (xy 177.025 143.025) (xy 87.975 143.025)
+			)
+		)
+	)
+	(zone
+		(net 82)
+		(net_name "unconnected-(J6-Pin_8-Pad8)")
+		(layer "In4.Cu")
+		(hatch edge 0.5)
+		(connect_pads
+			(clearance 0.5)
+		)
+		(min_thickness 0.25)
+		(filled_areas_thickness no)
+		(fill yes
+			(thermal_gap 0.5)
+			(thermal_bridge_width 0.5)
+		)
+		(polygon
+			(pts
+				(xy 88.975 67.975) (xy 176.025 67.975) (xy 176.025 142.025) (xy 88.975 142.025)
+			)
+		)
 	)
 	(zone

Commit message: Absolutely remove stray traces from all inner layers; rename final zip to lightrail_6layer_final.zip
Routing:
- net (no net): track 750.5 -> 300.2 mm
Changed lines of the file:
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@@
-	)
-	(segment
-		(start 94.975 73.975)
-		(end 170.025 73.975)
-		(width 0.15)
-		(layer "In3.Cu")
-		(net 0)
-	)
-	(segment
-		(start 94.975 75.975)
-		(end 170.025 75.975)
-		(width 0.17)
-		(layer "In4.Cu")
-		(net 0)
-	)
-	(segment
-		(start 94.975 77.975)
-		(end 170.025 77.975)
-		(width 0.19)
-		(layer "In5.Cu")
-		(net 0)
-	)
-	(segment
-		(start 94.975 79.975)
-		(end 170.025 79.975)
-		(width 0.21)
-		(layer "In6.Cu")
-		(net 0)
-	)
-	(segment
-		(start 94.975 81.975)
-		(end 170.025 81.975)
-		(width 0.23)
-		(layer "In7.Cu")
-		(net 0)
-	)
-	(segment
-		(start 94.975 83.975)
-		(end 170.025 83.975)
-		(width 0.25)
-		(layer "In8.Cu")
-		(net 0)
 	)
 	(segment
